Commit message: turtletests

File: first_robot/src/urdf/robot.urdf (robot description, URDF)
Before this commit: robot first_robot, 5 links, 4 joints
Links:
- link BL_wheel: geometry collision cylinder length=0.1 radius=0.1; visual cylinder length=0.1 radius=0.1
- link BR_wheel: geometry collision cylinder length=0.1 radius=0.1; visual cylinder length=0.1 radius=0.1
- link FL_wheel: geometry collision cylinder length=0.1 radius=0.1; visual cylinder length=0.1 radius=0.1
- link FR_wheel: geometry collision cylinder length=0.1 radius=0.1; visual cylinder length=0.1 radius=0.1
- link main_link: geometry collision box size=0.8 0.8 0.1; visual box size=0.8 0.8 0.1
